File: kicad-v2.0/ICanSolder.kicad_pcb (KiCad board)
At the start: 2 copper layers, 40 x 48.2 mm, 7 parts

Commit message: added version number for license
Other:
- board text added: "CC-BY-SA 4.0"
- board text added: "I can solder"
- board text removed: "CC-BY-SA"
- board text removed: "I Can Solder"

Commit message: generated ibom
Parts:
- removed REF**: MountingHole_2.2mm_M2_DIN965_Pad, MountingHole:MountingHole_2.2mm_M2_DIN965_Pad
- removed the Ref** at (122.0, 116.5)
- added H1: MountingHole_Pad, MountingHole:MountingHole_2.2mm_M2_DIN965_Pad, F.Cu at (181.0, 98.0)
Other:
- board text added: "+"
Changed lines of the file:
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@@
   (general
     (thickness 1.6)
-    (drawings 4)
+    (drawings 8)
     (tracks 6)
     (zones 0)
-    (modules 7)
+    (modules 6)
     (nets 3)
   )
@@
     (add_net VCC)
   )
+  (module MountingHole:MountingHole_2.2mm_M2_DIN965_Pad (layer F.Cu)
+    (at 180.962489 98)
+    (descr "Mounting Hole 2.2mm, M2, DIN965")
+    (tags "mounting hole 2.2mm m2 din965")
+    (attr virtual)
+    (fp_text reference H1 (at 0 -2.9) (layer F.SilkS) hide
+      (effects (font (size 1 1) (thickness 0.15)))
+    )
+    (fp_text value MountingHole_Pad (at 0 2.9) (layer F.Fab)
+      (effects (font (size 1 1) (thickness 0.15)))
+    )
+    (fp_circle (center 0 0) (end 2.15 0) (layer F.CrtYd) (width 0.05))
+    (fp_circle (center 0 0) (end 1.9 0) (layer Cmts.User) (width 0.15))
+    (fp_text user %R (at 0.3 0) (layer F.Fab)
+      (effects (font (size 1 1) (thickness 0.15)))
+    )
+    (pad 1 thru_hole circle (at 0 0) (size 3.8 3.8) (drill 2.2) (layers *.Cu *.Mask)
+      (net 1 GND))
+  )
   (module Binary-Kitchen:binary_kitchen_logo_prepared (layer F.Cu)
     (at 180.5 120.5)
+    (attr virtual)
     (fp_text reference Ref** (at 0 0) (layer F.SilkS) hide
       (effects (font (size 1.27 1.27) (thickness 0.15)))
@@
       (xy 0.755439 16.891) (xy 18.105545 16.891) (xy 18.186189 16.980111)) (layer B.Mask) (width 0.01))
   )
-  (module MountingHole:MountingHole_2.2mm_M2_DIN965_Pad (layer F.Cu)
-    (at 181 98.2)
-    (descr "Mounting Hole 2.2mm, M2, DIN965")
-    (tags "mounting hole 2.2mm m2 din965")
-    (attr virtual)
-    (fp_text reference REF** (at 0 -2.9) (layer F.SilkS) hide
-      (effects (font (size 1 1) (thickness 0.15)))
-    )
-    (fp_text value MountingHole_2.2mm_M2_DIN965_Pad (at 0 2.9) (layer F.Fab)
-      (effects (font (size 1 1) (thickness 0.15)))
-    )
-    (fp_circle (center 0 0) (end 1.9 0) (layer Cmts.User) (width 0.15))
-    (fp_circle (center 0 0) (end 2.15 0) (layer F.CrtYd) (width 0.05))
-    (fp_text user %R (at 0.3 0) (layer F.Fab)
-      (effects (font (size 1 1) (thickness 0.15)))
-    )
-    (pad 1 thru_hole circle (at 0 0) (size 3.8 3.8) (drill 2.2) (layers *.Cu *.Mask))
-  )
   (module LED_THT:LED_D5.0mm_Clear (layer F.Cu)
     (at 166.5 108)
@@
       (effects (font (size 1 1) (thickness 0.15)))
     )
-    (fp_text value LED (at 1.27 3.96) (layer F.Fab)
+    (fp_text value LED (at 1.27 3.96) (layer F.Fab) hide
       (effects (font (size 1 1) (thickness 0.15)))
     )
@@
     )
   )
-  (module Binary-Kitchen:binary_kitchen_logo_prepared (layer F.Cu)
-    (at 122 116.5)
-    (fp_text reference Ref** (at 0 0) (layer F.SilkS) hide
-      (effects (font (size 1.27 1.27) (thickness 0.15)))
-    )
-    (fp_text value Val** (at 0 0) (layer F.SilkS) hide
-      (effects (font (size 1.27 1.27) (thickness 0.15)))
-    )
-  )
   (module LED_THT:LED_D5.0mm_Clear (layer F.Cu)
     (at 192 108)
@@
       (effects (font (size 1 1) (thickness 0.15)))
     )
-    (fp_text value LED (at 1.27 3.96) (layer F.Fab)
+    (fp_text value LED (at 1.27 3.96) (layer F.Fab) hide
       (effects (font (size 1 1) (thickness 0.15)))
     )
@@
       (effects (font (size 1 1) (thickness 0.15)))
     )
-    (fp_text value LED (at 1.27 3.96) (layer F.Fab)
+    (fp_text value LED (at 1.27 3.96) (layer F.Fab) hide
       (effects (font (size 1 1) (thickness 0.15)))
     )
@@
     (descr "20MM (CR2032) COIN CELL BATTERY HOLDER - PTH")
     (tags "20MM (CR2032) COIN CELL BATTERY HOLDER - PTH")
-    (attr virtual)
     (fp_text reference BT1 (at -1.5 0 -90) (layer B.SilkS) hide
       (effects (font (size 0.6096 0.6096) (thickness 0.127)) (justify mirror))
     )
-    (fp_text value Battery_Cell (at 0 0 -90) (layer B.SilkS)
+    (fp_text value Battery_Cell (at 0 0 -90) (layer B.SilkS) hide
       (effects (font (size 0.6096 0.6096) (thickness 0.127)) (justify mirror))
     )
@@
       (net 2 VCC) (solder_mask_margin 0.1016))
   )
-  (gr_text "CC-BY-SA 4.0" (at 189.5 129.5) (layer B.SilkS)
+  (gr_text + (at 191.3 115.4) (layer B.SilkS)
+    (effects (font (size 0.5 0.5) (thickness 0.125)) (justify mirror))
+  )
+  (gr_text + (at 194.5 109.35) (layer B.SilkS)
+    (effects (font (size 0.5 0.5) (thickness 0.125)) (justify mirror))
+  )
+  (gr_text + (at 169 109.35) (layer B.SilkS)
+    (effects (font (size 0.5 0.5) (thickness 0.125)) (justify mirror))
+  )
+  (gr_text + (at 182.5 131.35) (layer B.SilkS)
+    (effects (font (size 0.5 0.5) (thickness 0.125)) (justify mirror))
+  )
+  (gr_text "CC-BY-SA 4.0" (at 189.4 129.5) (layer B.SilkS)
     (effects (font (size 0.8 0.8) (thickness 0.11)) (justify mirror))
   )
-  (gr_text "Binary Kitchen" (at 189.6 127.85) (layer B.SilkS)
+  (gr_text "Binary Kitchen" (at 189.5 127.85) (layer B.SilkS)
     (effects (font (size 0.8 0.8) (thickness 0.11)) (justify mirror))
   )
